File: data/kicad/TXJ1.kicad_pcb (KiCad board)
At the start: 2 copper layers, 23 x 11 mm, 16 parts

Commit message: Step 2: CB1D options, SB1R via drill, TXJ1 pads, fab-floor rules, finishes (KiCad 9: 5 boards, 0 errors / 0 unconnected)
- SB1R: via drill 0.4 mm (was 0.8 = no annular ring in the KiCad files and the PTH drill files); QB transfer nets QB_T1/QB_T2; Gerbers SB1R_QA_v2 / SB1R_QB_v2, old marked superseded; sbq sims unchanged (0 numbers moved)
- TXJ1: AWG12 pads 3.8 mm (edge distance 0.6 mm); Gerbers TXJ1_v2
- CB1D: RJB10 0R fitted on JB.10, RJ5/RJ6 DNP grounds for JTR.5/.6 (61 parts, 44/44 nets); Gerbers CB1D_B2; wiring alias JB10_VCM
- dru_gen: conservative Advanced Circuits / TTM floor (UNVERIFIED), SB1R keys; no ENIG near the coil/receivers (immersion silver / HASL); docs/design/FAB_RULES.md
- make kicad-drc covers CB1D, LB1, TXJ1, SB1R-QA/QB; regress 42 pass; CORRECTIONS, DESIGN_STATE, OPEN_ITEMS 23/25-27, ASSUMPTIONS 31

Co-Authored-By: Claude Sonnet 5.5 <noreply@anthropic.com>
Claude-Session: https://claude.ai/code/session_01T7iU5pGiBfkKRBbe2JcTJx
Changed lines of the file:
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@@
   (paper "A4")
   (layers (0 "F.Cu" signal) (31 "B.Cu" signal) (36 "B.SilkS" user "B.Silkscreen") (37 "F.SilkS" user "F.Silkscreen") (38 "B.Mask" user) (39 "F.Mask" user) (44 "Edge.Cuts" user))
-  (setup (pad_to_mask_clearance 0.05) (stackup (layer "F.Cu" (type "copper") (thickness 0.07)) (layer "dielectric 1" (type "core") (thickness 1.46)) (layer "B.Cu" (type "copper") (thickness 0.07)) (copper_finish "ENIG")))
+  (setup (pad_to_mask_clearance 0.05) (stackup (layer "F.Cu" (type "copper") (thickness 0.07)) (layer "dielectric 1" (type "core") (thickness 1.46)) (layer "B.Cu" (type "copper") (thickness 0.07)) (copper_finish "Immersion silver")))
   (net 0 "")
   (net 1 "TX_A")
@@
   (footprint "TXJ1:PTH" (layer "F.Cu") (at 97.000 103.000) (property "Reference" "TAPA" (at 0 -2.4) (layer "F.SilkS")) (pad "1" thru_hole circle (at 0 0) (size 2.0 2.0) (drill 1.0) (layers "*.Cu" "*.Mask") (net 1 "TX_A")))
   (footprint "TXJ1:PTH" (layer "F.Cu") (at 97.000 97.000) (property "Reference" "TAPB" (at 0 -2.4) (layer "F.SilkS")) (pad "1" thru_hole circle (at 0 0) (size 2.0 2.0) (drill 1.0) (layers "*.Cu" "*.Mask") (net 2 "TX_B")))
-  (footprint "TXJ1:PTH" (layer "F.Cu") (at 115.500 103.000) (property "Reference" "A12" (at 0 -2.4) (layer "F.SilkS")) (pad "1" thru_hole circle (at 0 0) (size 4.2 4.2) (drill 2.6) (layers "*.Cu" "*.Mask") (net 1 "TX_A")))
-  (footprint "TXJ1:PTH" (layer "F.Cu") (at 115.500 97.000) (property "Reference" "B12" (at 0 -2.4) (layer "F.SilkS")) (pad "1" thru_hole circle (at 0 0) (size 4.2 4.2) (drill 2.6) (layers "*.Cu" "*.Mask") (net 2 "TX_B")))
+  (footprint "TXJ1:PTH" (layer "F.Cu") (at 115.500 103.000) (property "Reference" "A12" (at 0 -2.4) (layer "F.SilkS")) (pad "1" thru_hole circle (at 0 0) (size 3.8 3.8) (drill 2.6) (layers "*.Cu" "*.Mask") (net 1 "TX_A")))
+  (footprint "TXJ1:PTH" (layer "F.Cu") (at 115.500 97.000) (property "Reference" "B12" (at 0 -2.4) (layer "F.SilkS")) (pad "1" thru_hole circle (at 0 0) (size 3.8 3.8) (drill 2.6) (layers "*.Cu" "*.Mask") (net 2 "TX_B")))
   (segment (start 97.000 103.000) (end 115.500 103.000) (width 3.0) (layer "F.Cu") (net 1))
   (segment (start 97.000 97.000) (end 115.500 97.000) (width 3.0) (layer "B.Cu") (net 2))
