File: data/kicad/PF233-LB1_routed.kicad_pcb (KiCad board)
At the start: 4 copper layers, 78 x 77.2 mm, 81 parts, among them U1 74AHCT1G125

Commit message: Step 5: datasheets and fabricator sheets (vendor-derived floor, verified parts, PB1R 9-can bank, Gerber edge read-back)
- Fab floor from AdvancedPCB / TTM pages (docs/design/FAB_RULES_VERIFIED.md, U-FAB-RULES closed): clearance 0.16,
  component-PTH ring 0.18 / hole 0.46, drill-copper 0.26, drill-drill 0.41, every rule (severity error).
  CB1D JA/JB and HB2 TO-92 pads 1.02 mm; route_fix merges close same-net vias (CB1D, LB1).
- Parts from manufacturer PDFs (docs/design/DATASHEET_LOG.md): PB1R bulk 9 x Panasonic EEHZC1H101P
  (the 150 uF / 50 V polymer-Ta was not found; bank stays 900 uF, on-time table unchanged), PB1R re-placed
  with the Kelvin/comparator cluster pinned (pulse path 4.9 mohm, spike 7.5 V, ground ref 15.5 mV unchanged);
  SMCJ30A (SMCJ33A clamps 53.3 V > 50 V parts), Si4401FDY, BZT52C15, Bourns SF-1206S500-2 (new 1206 land),
  DRV5023BIQLPG, CRCW2512 500 V, OPA2365/OPA2211/LM393/CD74HC4051 checked. ES3J 600 V kept as a WATCH.
- U-DS-PARTS split into groups; open: TXDRIVE, OKI, PACK, BAV199, HVTERM. U-COLD-BOOTSTRAP closed.
- Controls retargeted to fixture folders (12/12). Netlist date fixed (data changed daily).
- Gerber planes from gerber_out.py ran into the notch and to 0.1 mm of the edge since r1 (found by the
  independent review): fixed, and gerber_edge_check.py reads every copper layer back.
- New Gerber sets CB1D_B3, LB1_v5, PB1R_v2; old sets marked SUPERSEDED.
- Findings for the owner: aluminium cans ~0.5 x a 1 g nugget (OPEN_ITEMS 34), OPA2365 capacitive load (30),
  OPA2211 input range on 5 V (31), Hall magnet spread (32).
- Strict regress 55 PASS / 0 FAIL / 0 SKIP; sign-off 44 PASS / 0 FAIL / 0 SKIP / 19 UNVERIFIED.

Co-Authored-By: Claude Opus 5.5 <noreply@anthropic.com>
Claude-Session: https://claude.ai/code/session_015VKhZtgEAWnezB2NDY75VV
Routing:
- net GND: track 183.3 -> 183.9 mm, vias 80 -> 79
Changed lines of the file:
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@@
   (segment (start 132.8620 112.1610) (end 132.7500 112.6500) (width 0.2) (layer "F.Cu") (net 66))
   (segment (start 132.7500 112.6500) (end 132.8620 112.1610) (width 0.2) (layer "F.Cu") (net 66))
+  (segment (start 107.4000 99.9000) (end 107.4000 100.5000) (width 0.4) (layer "F.Cu") (net 2))
   (via (at 112.5000 97.2000) (size 0.6) (drill 0.3) (layers "F.Cu" "B.Cu") (net 2))
   (via (at 109.2000 91.5000) (size 0.6) (drill 0.3) (layers "F.Cu" "B.Cu") (net 2))
@@
   (via (at 104.2500 102.6000) (size 0.6) (drill 0.3) (layers "F.Cu" "B.Cu") (net 2))
   (via (at 107.4000 100.5000) (size 0.6) (drill 0.3) (layers "F.Cu" "B.Cu") (net 2))
-  (via (at 107.4000 99.9000) (size 0.6) (drill 0.3) (layers "F.Cu" "B.Cu") (net 2))
   (via (at 108.3000 96.9000) (size 0.6) (drill 0.3) (layers "F.Cu" "B.Cu") (net 2))
   (via (at 108.3000 94.9500) (size 0.6) (drill 0.3) (layers "F.Cu" "B.Cu") (net 2))
