File: data/kicad/PF233-PB1R_placed.kicad_pcb (KiCad board)
At the start: 4 copper layers, 70 x 70 mm, 42 parts, among them M12 12 V 1.5 A switching module, Q1A 650V SJ 95mR, Q1B 650V SJ 95mR, U1 TC4420, U3 LM393

Commit message: WIP stage 5: B3/B5/B6/B8 closed in blockers.json, B7 narrowed to HVTERM, B12 opened; cap-v18 pipeline step (cap was not regenerated on a fresh work/); upper_check septum joint by voxels; curated STLs refreshed (U6 dock for the real MT60, septum lap segments, canonical face order); DESIGN_STATE stress counts
Co-Authored-By: Claude Opus 5.5 <noreply@anthropic.com>
Claude-Session: https://claude.ai/code/session_01FX4DWSYYjMCFGGA6gmha65
Parts:
- M12: value 12 V 1.5 A switching module -> 12 V 1.0 A switching module
Changed lines of the file:
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@@
   (footprint "Converter_DCDC:Converter_DCDC_Murata_OKI-78SR_Horizontal" (layer "F.Cu") (at 114.0000 73.0000)
     (property "Reference" "M12" (at 0 -2.5 0) (layer "F.SilkS") (effects (font (size 0.8 0.8) (thickness 0.12))))
-    (property "Value" "12 V 1.5 A switching module" (at 0 2.5 0) (layer "F.Fab") (effects (font (size 0.8 0.8) (thickness 0.12))))
+    (property "Value" "12 V 1.0 A switching module" (at 0 2.5 0) (layer "F.Fab") (effects (font (size 0.8 0.8) (thickness 0.12))))
     (attr through_hole)
     (model "${KIPRJMOD}/3dmodels/PF233_OKI3.wrl" (offset (xyz 0 0 0)) (scale (xyz 0.3937 0.3937 0.3937)) (rotate (xyz 0 0 0)))
