File: data/kicad/PF233-HB2_routed.kicad_pcb (KiCad board)
At the start: 4 copper layers, 24 x 38 mm, 10 parts

Commit message: WIP (NOT signed off): data published by the first close-out sign-off run, which had 5 FAIL (CB1D-C2 / AU1 fine-pitch clearance); superseded by the rerun in progress
Co-Authored-By: Claude Opus 5.5 <noreply@anthropic.com>
Claude-Session: https://claude.ai/code/session_01FX4DWSYYjMCFGGA6gmha65
Parts:
- added JAU: Lead to AU1: AUD_LINK, GND, Connector:SolderPad_2x_P5.08mm, F.Cu at (95.0, 106.0)
- moved RD3 2.00 mm to (98.0, 109.0)
Connections:
- JH pad 5: JH5_NC -> AUD_LINK
Routing:
- net AUD_LINK: track 0.00 -> 10.3 mm
- net DP3: track 18.0 -> 21.4 mm
- net P3V3: track 39.9 -> 42.1 mm, vias 3 -> 2
- net TRIG: track 31.0 -> 28.9 mm, vias 0 -> 2
- net SHIELD: track 9.02 -> 11.0 mm

Commit message: Close-out of the output modes / audio / gyro integration: sign-off 76 PASS / 0 FAIL / 4 UNVERIFIED, strict regress 114 / 0, release controls 12 / 12, publish 0 stale
AU1 (36 x 60, 8 layers, gyro moved from CB1D) routed 38 / 38, CB1D-C2 46 / 46, both exact DRC 0 / 0; PB1R-v5 AWG12 solder holes; PM2-B, HB2-B; superseded Gerber sets marked.
Tooling now default: exact-geometry DRC, router fine-pitch keep-out / neck-down / per-board grid, local repair, round checkpoints, non-destructive reset,
interface check, AU1 3-D models with gull-wing leads, counted HV check; pad check traced by the pipeline; process-guard regress row; PROCESS.md / CLAUDE.md / handoff updated.

Co-Authored-By: Claude Opus 5.5 <noreply@anthropic.com>
Claude-Session: https://claude.ai/code/session_01FX4DWSYYjMCFGGA6gmha65
Parts:
- removed the JDIAL at (106.0, 90.0)
- removed the JH at (93.0, 94.0)
- added JDIAL: Dial: COM P1 P2 P3 P4 (4-pos rotary, top housing), Connector:Wire_pads_1x5_P2.54mm, F.Cu at (106.0, 90.0)
- added JH: Signal cord to the head: +3V3 GND TRIG DIAL - - SHLD, Connector:Wire_pads_1x7_P2.54mm, F.Cu at (93.0, 94.0)
Changed lines of the file:
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@@
   (net 10 "SHIELD")
   (net 11 "TRIG")
-  (footprint "Connector:Pin_header_1x7_P2.54mm" (layer "F.Cu") (at 93.0000 94.0000)
+  (footprint "Connector:Wire_pads_1x7_P2.54mm" (layer "F.Cu") (at 93.0000 94.0000)
     (property "Reference" "JH" (at 0 -2.5 0) (layer "F.SilkS") (effects (font (size 0.8 0.8) (thickness 0.12))))
     (property "Value" "Signal cord to the head: +3V3 GND TRIG DIAL - - SHLD" (at 0 2.5 0) (layer "F.Fab") (effects (font (size 0.8 0.8) (thickness 0.12))))
@@
     (pad "2" smd roundrect (at 0.825 0.000) (size 0.800 0.950) (layers "F.Cu" "F.Paste" "F.Mask") (net 11 "TRIG"))
   )
-  (footprint "Connector:Pin_header_1x5_P2.54mm" (layer "F.Cu") (at 106.0000 90.0000)
+  (footprint "Connector:Wire_pads_1x5_P2.54mm" (layer "F.Cu") (at 106.0000 90.0000)
     (property "Reference" "JDIAL" (at 0 -2.5 0) (layer "F.SilkS") (effects (font (size 0.8 0.8) (thickness 0.12))))
     (property "Value" "Dial: COM P1 P2 P3 P4 (4-pos rotary, top housing)" (at 0 2.5 0) (layer "F.Fab") (effects (font (size 0.8 0.8) (thickness 0.12))))
