File: data/kicad/sch_functional/PF233-AB1A_functional.kicad_sch (KiCad schematic)
At the start: 56 parts, among them J1 Antenna harness 8p solder pad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, J2 Main-board 2x6 1.27mm header, SW1 74LVC1G66, SW2 74LVC1G66, SW3 74LVC1G66, U1 OPA2211, U2 OPA2211

Commit message: Stage A: pipeline graph re-learned with the AB1 steps (58 steps), sign-off 67 PASS / 0 FAIL, controls updated for 11 boards, published AB1 results and Gerbers
Co-Authored-By: Claude Sonnet 5.5 <noreply@anthropic.com>
Claude-Session: https://claude.ai/code/session_015VKhZtgEAWnezB2NDY75VV
Parts:
- removed CAV1, CAV2, CAV3, CDV1, CDV2, CDV3: 100n, Capacitor_SMD:C_0402_1005Metric, symbol PF233F:C_H
- removed CRF1, CRF2, CRF3: 10u, Capacitor_SMD:C_0805_2012Metric, symbol PF233F:C_H
- removed CRI, CRN, CRO: 1u, Capacitor_SMD:C_0603_1608Metric, symbol PF233F:C_H
- removed UA2, UA3: ADS8860, Package_SO:MSOP-10_3x3mm_P0.5mm, symbol PF233F:BOX_ADS8860
- removed UR: REF5041, Package_SO:MSOP-8_3x3mm_P0.65mm, symbol PF233F:BOX_REF5041
- added CRC: 100n, Capacitor_SMD:C_0402_1005Metric, symbol PF233F:C_H
- added CRF, CRG, CVC, CVL: 1u, Capacitor_SMD:C_0402_1005Metric, symbol PF233F:C_H
- RD1, RD2: value 10k -> 100k
- UA1: value ADS8860 -> AD7389-4; footprint Package_SO:MSOP-10_3x3mm_P0.5mm -> Package_CSP:LFCSP-24-1EP_4x4mm_P0.5mm_EP2.65x2.65mm; symbol PF233F:BOX_ADS8860 -> PF233F:BOX_AD7389
Connections:
- net +3V3D: now also UA1.2 (VLOGIC), UA1.4 (VCC33), CVC.1, CVL.1; no longer UA1.9 (DVDD)
- net +5VA: no longer UA1.2 (AVDD)
- net ADCIN_GX: now also UA1.13 (AINA+); no longer UA1.3 (AINP)
- net ADCIN_GY: now also UA1.11 (AINB+)
- net ADCIN_X8: now also UA1.9 (AINC+)
- net CS: now also UA1.18 (CS); no longer UA1.6 (CS)
- net GND: now also UA1.1 (GND), UA1.14 (GND), UA1.16 (GND), UA1.21 (SDI), UA1.25 (EP), CRC.2, CRF.2, CRG.2, CVC.2, CVL.2; no longer UA1.10 (GND2), UA1.4 (AINN)
- net SCLK: now also UA1.22 (SCLK); no longer UA1.8 (SCLK)
- net SDO1: now also UA1.19 (SDOA); no longer UA1.7 (SDO)
- net SDO2: now also UA1.20 (SDOB)
- net VCM: now also UA1.10 (AINB-), UA1.12 (AINA-), UA1.6 (AIND-), UA1.7 (AIND+), UA1.8 (AINC-)
- net VREF: no longer UA1.1 (REF)
- net VREF_RAW: now also UA1.17 (REFOUT), CRF.1
- net SDO3: no longer names the net of J2.9
- new net REFCAP: CRC.1, UA1.15 (REFCAP)
- new net REGCAP: CRG.1, UA1.3 (REGCAP)
- no-connect marks 4 -> 3
Other:
- note added: "7 Quad simultaneous ADC"
- note added: "Non-inverting gain stage: RG1 to VCM, RF1 || CF1 feedback; OUT_GX -> RAAF1 / CAAF1 anti-alias -> ADCIN_GX -> UA1 input pair 1 (AD7389-4, differential: AIN+ = ADCIN_GX, AIN- = VCM)."
- note added: "Non-inverting gain stage: RG2 to VCM, RF2 || CF2 feedback; OUT_GY -> RAAF2 / CAAF2 anti-alias -> ADCIN_GY -> UA1 input pair 2 (AD7389-4, differential: AIN+ = ADCIN_GY, AIN- = VCM)."
- note added: "Non-inverting gain stage: RG3 to VCM, RF3 || CF3 feedback; OUT_X8 -> RAAF3 / CAAF3 anti-alias -> ADCIN_X8 -> UA1 input pair 3 (AD7389-4, differential: AIN+ = ADCIN_X8, AIN- = VCM)."
- note added: "PF233-AB1A: AB1A receive analog board: 3 channels (GX, GY, X8), blanking, gain, 16-bit quad ADC (AD7389-4)"
- note added: "The shared AD7389-4 is in block 7."
- note added: "UA1 AD7389-4 (16-bit, 2 MSPS, four differential inputs, internal reference): inputs ADCIN_* with VCM; unused pairs are parked on VCM."
- note added: "UA1 REFOUT (internal 2.5 V) -> VREF_RAW (CRF 1 uF); RD1 / RD2 (100 k) divide it to VCM_DIV (1.25 V) -> UB (OPA2365) half B -> VCM (CVM); UB half A is parked as a follower."
- note added: "VCC and VLOGIC from +3V3D (CVC, CVL 1 uF), REGCAP (CRG), REFCAP (CRC), REFOUT (CRF). 2-wire readout: SDOA (channels A then C) to J2 SDO1, SDOB to J2 SDO2; SDI tied to GND; CS starts a conversion."
- note removed: "Non-inverting gain stage: RG1 to VCM, RF1 || CF1 feedback; OUT_GX -> RAAF1 / CAAF1 anti-alias -> ADCIN_GX -> UA1 (ADS8860, 16-bit SAR; REF = VREF with CRF1)."
- note removed: "Non-inverting gain stage: RG2 to VCM, RF2 || CF2 feedback; OUT_GY -> RAAF2 / CAAF2 anti-alias -> ADCIN_GY -> UA2 (ADS8860, 16-bit SAR; REF = VREF with CRF2)."
- note removed: "Non-inverting gain stage: RG3 to VCM, RF3 || CF3 feedback; OUT_X8 -> RAAF3 / CAAF3 anti-alias -> ADCIN_X8 -> UA3 (ADS8860, 16-bit SAR; REF = VREF with CRF3)."
- note removed: "PF233-AB1A: AB1A receive analog board: 3 channels (GX, GY, X8), blanking, gain, 16-bit ADC"
- note removed: "SPI: SCLK / CS from the main board, SDO1 back."
- note removed: "SPI: SCLK / CS from the main board, SDO2 back."
- note removed: "SPI: SCLK / CS from the main board, SDO3 back."
- note removed: "UR (REF5041) -> VREF_RAW (CRI / CRO / CRN) -> UB (OPA2365) buffers VREF for the ADCs; RD1 / RD2 / CDF divide VREF_RAW to VCM_DIV -> UB other half -> VCM (CVM)."
- moved on the sheet: CAAF2, CAAF3, CB1, CBD, CDF, CF2, CF3, CO1, CO2, CSW2, CSW3, CVM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

Commit message: WIP: B5 link check, B6 readout model, B7 datasheets, B8 BOM/PnP + potting + septum lap, B9 rip-up router + drive option, solid_union cache, B3 rows (untested in pipeline)
Co-Authored-By: Claude Opus 5.5 <noreply@anthropic.com>
Claude-Session: https://claude.ai/code/session_01FX4DWSYYjMCFGGA6gmha65
Parts:
- UA1: footprint Package_CSP:LFCSP-24-1EP_4x4mm_P0.5mm_EP2.65x2.65mm -> Package_CSP:CP-24-25_ADI_LFCSP-24-1EP_4x4mm_P0.5mm_EP0.61x0.61mm
Changed lines of the file:
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@@
     (property "Reference" "UA1" (at 58.420 331.810 0) (effects (font (size 1.27 1.27))))
     (property "Value" "AD7389-4" (at 58.420 388.120 0) (effects (font (size 1.0 1.0))))
-    (property "Footprint" "Package_CSP:LFCSP-24-1EP_4x4mm_P0.5mm_EP2.65x2.65mm" (at 58.420 363.220 0) (effects (font (size 1.27 1.27)) hide))
+    (property "Footprint" "Package_CSP:CP-24-25_ADI_LFCSP-24-1EP_4x4mm_P0.5mm_EP0.61x0.61mm" (at 58.420 363.220 0) (effects (font (size 1.27 1.27)) hide))
     (pin "13")
     (pin "12")
