File: data/kicad/sch_functional/PF233-LB1_functional.kicad_sch (KiCad schematic)
At the start: 81 parts, among them U1 74AHCT1G125

Commit message: WIP: sign-off re-run outputs (publish in progress)
Co-Authored-By: Claude Opus 5.5 <noreply@anthropic.com>
Claude-Session: https://claude.ai/code/session_01FX4DWSYYjMCFGGA6gmha65
Parts:
- added RSC: 33R, Resistor_SMD:R_0603_1608Metric, symbol PF233F:R_H
- added U2: 74AHCT1G125, Package_TO_SOT_SMD:SOT-23-5, symbol PF233F:BOX_SOT23-5
- JLB: value to CB1D: +5V, LED_IN, GND, GND -> to CB1D: +5V, LED_IN, LED_CLK, GND
- LD1, LD10, LD11, LD12, LD13, LD14, LD15, LD16, LD17, LD18, LD19, LD2, LD20, LD21, LD22, LD23, LD24, LD25, LD26, LD27, LD28, LD29, LD3, LD30, LD31, LD32, LD33, LD34, LD35, LD36, LD37, LD38, LD39, LD4, LD40, LD41, LD42, LD43, LD44, LD45, LD46, LD47, LD48, LD49, LD5, LD50, LD51, LD52, LD53, LD54, LD55, LD56, LD57, LD58, LD59, LD6, LD60, LD61, LD62, LD63, LD64, LD65, LD66, LD7, LD8, LD9: value SK6812 MINI-E RGB -> SK9822-EC20 RGB; footprint LED_SMD:LED_SK6812MINI-E_3.2x2.8mm -> PF233:LED_SK9822-EC20_2.0x2.0mm; symbol PF233F:BOX_LED2020 -> PF233F:BOX_SK9822EC20
Connections:
- net +5V: now also LD1.5 (VDD), LD10.5 (VDD), LD11.5 (VDD), LD12.5 (VDD), LD13.5 (VDD), LD14.5 (VDD), LD15.5 (VDD), LD16.5 (VDD), LD17.5 (VDD), LD18.5 (VDD), LD19.5 (VDD), LD2.5 (VDD), LD20.5 (VDD), LD21.5 (VDD), LD22.5 (VDD), LD23.5 (VDD), LD24.5 (VDD), LD25.5 (VDD), LD26.5 (VDD), LD27.5 (VDD), LD28.5 (VDD), LD29.5 (VDD), LD3.5 (VDD), LD30.5 (VDD), LD31.5 (VDD), LD32.5 (VDD), LD33.5 (VDD), LD34.5 (VDD), LD35.5 (VDD), LD36.5 (VDD), LD37.5 (VDD), LD38.5 (VDD), LD39.5 (VDD), LD4.5 (VDD), LD40.5 (VDD), LD41.5 (VDD), LD42.5 (VDD), LD43.5 (VDD), LD44.5 (VDD), LD45.5 (VDD), LD46.5 (VDD), LD47.5 (VDD), LD48.5 (VDD), LD49.5 (VDD), LD5.5 (VDD), LD50.5 (VDD), LD51.5 (VDD), LD52.5 (VDD), LD53.5 (VDD), LD54.5 (VDD), LD55.5 (VDD), LD56.5 (VDD), LD57.5 (VDD), LD58.5 (VDD), LD59.5 (VDD), LD6.5 (VDD), LD60.5 (VDD), LD61.5 (VDD), LD62.5 (VDD), LD63.5 (VDD), LD64.5 (VDD), LD65.5 (VDD), LD66.5 (VDD), LD7.5 (VDD), LD8.5 (VDD), LD9.5 (VDD), U2.5 (VCC); no longer LD1.1 (VDD), LD10.1 (VDD), LD11.1 (VDD), LD12.1 (VDD), LD13.1 (VDD), LD14.1 (VDD), LD15.1 (VDD), LD16.1 (VDD), LD17.1 (VDD), LD18.1 (VDD), LD19.1 (VDD), LD2.1 (VDD), LD20.1 (VDD), LD21.1 (VDD), LD22.1 (VDD), LD23.1 (VDD), LD24.1 (VDD), LD25.1 (VDD), LD26.1 (VDD), LD27.1 (VDD), LD28.1 (VDD), LD29.1 (VDD), LD3.1 (VDD), LD30.1 (VDD), LD31.1 (VDD), LD32.1 (VDD), LD33.1 (VDD), LD34.1 (VDD), LD35.1 (VDD), LD36.1 (VDD), LD37.1 (VDD), LD38.1 (VDD), LD39.1 (VDD), LD4.1 (VDD), LD40.1 (VDD), LD41.1 (VDD), LD42.1 (VDD), LD43.1 (VDD), LD44.1 (VDD), LD45.1 (VDD), LD46.1 (VDD), LD47.1 (VDD), LD48.1 (VDD), LD49.1 (VDD), LD5.1 (VDD), LD50.1 (VDD), LD51.1 (VDD), LD52.1 (VDD), LD53.1 (VDD), LD54.1 (VDD), LD55.1 (VDD), LD56.1 (VDD), LD57.1 (VDD), LD58.1 (VDD), LD59.1 (VDD), LD6.1 (VDD), LD60.1 (VDD), LD61.1 (VDD), LD62.1 (VDD), LD63.1 (VDD), LD64.1 (VDD), LD65.1 (VDD), LD66.1 (VDD), LD7.1 (VDD), LD8.1 (VDD), LD9.1 (VDD)
- net GND: now also LD1.2 (GND), LD10.2 (GND), LD11.2 (GND), LD12.2 (GND), LD13.2 (GND), LD14.2 (GND), LD15.2 (GND), LD16.2 (GND), LD17.2 (GND), LD18.2 (GND), LD19.2 (GND), LD2.2 (GND), LD20.2 (GND), LD21.2 (GND), LD22.2 (GND), LD23.2 (GND), LD24.2 (GND), LD25.2 (GND), LD26.2 (GND), LD27.2 (GND), LD28.2 (GND), LD29.2 (GND), LD3.2 (GND), LD30.2 (GND), LD31.2 (GND), LD32.2 (GND), LD33.2 (GND), LD34.2 (GND), LD35.2 (GND), LD36.2 (GND), LD37.2 (GND), LD38.2 (GND), LD39.2 (GND), LD4.2 (GND), LD40.2 (GND), LD41.2 (GND), LD42.2 (GND), LD43.2 (GND), LD44.2 (GND), LD45.2 (GND), LD46.2 (GND), LD47.2 (GND), LD48.2 (GND), LD49.2 (GND), LD5.2 (GND), LD50.2 (GND), LD51.2 (GND), LD52.2 (GND), LD53.2 (GND), LD54.2 (GND), LD55.2 (GND), LD56.2 (GND), LD57.2 (GND), LD58.2 (GND), LD59.2 (GND), LD6.2 (GND), LD60.2 (GND), LD61.2 (GND), LD62.2 (GND), LD63.2 (GND), LD64.2 (GND), LD65.2 (GND), LD66.2 (GND), LD7.2 (GND), LD8.2 (GND), LD9.2 (GND), U2.1 (OE), U2.3 (GND); no longer JLB.3, LD1.3 (GND), LD10.3 (GND), LD11.3 (GND), LD12.3 (GND), LD13.3 (GND), LD14.3 (GND), LD15.3 (GND), LD16.3 (GND), LD17.3 (GND), LD18.3 (GND), LD19.3 (GND), LD2.3 (GND), LD20.3 (GND), LD21.3 (GND), LD22.3 (GND), LD23.3 (GND), LD24.3 (GND), LD25.3 (GND), LD26.3 (GND), LD27.3 (GND), LD28.3 (GND), LD29.3 (GND), LD3.3 (GND), LD30.3 (GND), LD31.3 (GND), LD32.3 (GND), LD33.3 (GND), LD34.3 (GND), LD35.3 (GND), LD36.3 (GND), LD37.3 (GND), LD38.3 (GND), LD39.3 (GND), LD4.3 (GND), LD40.3 (GND), LD41.3 (GND), LD42.3 (GND), LD43.3 (GND), LD44.3 (GND), LD45.3 (GND), LD46.3 (GND), LD47.3 (GND), LD48.3 (GND), LD49.3 (GND), LD5.3 (GND), LD50.3 (GND), LD51.3 (GND), LD52.3 (GND), LD53.3 (GND), LD54.3 (GND), LD55.3 (GND), LD56.3 (GND), LD57.3 (GND), LD58.3 (GND), LD59.3 (GND), LD6.3 (GND), LD60.3 (GND), LD61.3 (GND), LD62.3 (GND), LD63.3 (GND), LD64.3 (GND), LD65.3 (GND), LD66.3 (GND), LD7.3 (GND), LD8.3 (GND), LD9.3 (GND)
- net LD_D0: now also LD1.3 (SDI); no longer LD1.4 (DIN)
- net LD_D11: now also LD11.1 (SDO), LD12.3 (SDI); no longer LD11.2 (DOUT), LD12.4 (DIN)
- net LD_D22: now also LD22.1 (SDO), LD23.3 (SDI); no longer LD22.2 (DOUT), LD23.4 (DIN)
- net LD_D33: now also LD33.1 (SDO), LD34.3 (SDI); no longer LD33.2 (DOUT), LD34.4 (DIN)
- net LD_D44: now also LD44.1 (SDO), LD45.3 (SDI); no longer LD44.2 (DOUT), LD45.4 (DIN)
- net LD_D55: now also LD55.1 (SDO), LD56.3 (SDI); no longer LD55.2 (DOUT), LD56.4 (DIN)
- net LD_C24: now reaches LD25.4 (CKI)
- net LD_C24: now also LD24.6 (CKO); no longer LD24.2 (DOUT)
- net LD_C23: now reaches LD24.4 (CKI)
- net LD_C23: now also LD23.6 (CKO); no longer LD23.2 (DOUT)
- net LD_C31: now reaches LD32.4 (CKI)
- net LD_C31: now also LD31.6 (CKO); no longer LD31.2 (DOUT)
- net LD_C30: now reaches LD31.4 (CKI)
- net LD_C30: now also LD30.6 (CKO); no longer LD30.2 (DOUT)
- net LD_C61: now reaches LD62.4 (CKI)
- net LD_C61: now also LD61.6 (CKO); no longer LD61.2 (DOUT)
- net LD_C60: now reaches LD61.4 (CKI)
- net LD_C60: now also LD60.6 (CKO); no longer LD60.2 (DOUT)
- net LD_C57: now reaches LD58.4 (CKI)
- net LD_C57: now also LD57.6 (CKO); no longer LD57.2 (DOUT)
- net LD_C56: now reaches LD57.4 (CKI)
- net LD_C56: now also LD56.6 (CKO); no longer LD56.2 (DOUT)
- net LD_C29: now reaches LD30.4 (CKI)
- net LD_C29: now also LD29.6 (CKO); no longer LD29.2 (DOUT)
- net LD_C28: now reaches LD29.4 (CKI)
- net LD_C28: now also LD28.6 (CKO); no longer LD28.2 (DOUT)
- net LD_C26: now reaches LD27.4 (CKI)
- net LD_C26: now also LD26.6 (CKO); no longer LD26.2 (DOUT)
- net LD_C25: now reaches LD26.4 (CKI)
- net LD_C25: now also LD25.6 (CKO); no longer LD25.2 (DOUT)
- net LD_C38: now reaches LD39.4 (CKI)
- net LD_C38: now also LD38.6 (CKO); no longer LD38.2 (DOUT)
- net LD_C37: now reaches LD38.4 (CKI)
- net LD_C37: now also LD37.6 (CKO); no longer LD37.2 (DOUT)
- net LD_C13: now reaches LD14.4 (CKI)
- net LD_C13: now also LD13.6 (CKO); no longer LD13.2 (DOUT)
- net LD_C12: now reaches LD13.4 (CKI)
- net LD_C12: now also LD12.6 (CKO); no longer LD12.2 (DOUT)
- net LD_C43: now reaches LD44.4 (CKI)
- net LD_C43: now also LD43.6 (CKO); no longer LD43.2 (DOUT)
- net LD_C42: now reaches LD43.4 (CKI)
- net LD_C42: now also LD42.6 (CKO); no longer LD42.2 (DOUT)
- net LD_C27: now reaches LD28.4 (CKI)
- net LD_C27: now also LD27.6 (CKO); no longer LD27.2 (DOUT)
- net LD_C18: now reaches LD19.4 (CKI)
- net LD_C18: now also LD18.6 (CKO); no longer LD18.2 (DOUT)
- net LD_C17: now reaches LD18.4 (CKI)
- net LD_C17: now also LD17.6 (CKO); no longer LD17.2 (DOUT)
- net LD_C35: now reaches LD36.4 (CKI)
- net LD_C35: now also LD35.6 (CKO); no longer LD35.2 (DOUT)
- net LD_C34: now reaches LD35.4 (CKI)
- net LD_C34: now also LD34.6 (CKO); no longer LD34.2 (DOUT)
- net LD_C65: now reaches LD66.4 (CKI)
- net LD_C65: now also LD65.6 (CKO); no longer LD65.2 (DOUT)
- net LD_C64: now reaches LD65.4 (CKI)
- net LD_C64: now also LD64.6 (CKO); no longer LD64.2 (DOUT)
- net LD_C59: now reaches LD60.4 (CKI)
- net LD_C59: now also LD59.6 (CKO); no longer LD59.2 (DOUT)
- net LD_C9: now reaches LD10.4 (CKI)
- net LD_C9: now also LD9.6 (CKO); no longer LD9.2 (DOUT)
- net LD_C8: now reaches LD9.4 (CKI)
- net LD_C8: now also LD8.6 (CKO); no longer LD8.2 (DOUT)
- net LD_C15: now reaches LD16.4 (CKI)
- net LD_C15: now also LD15.6 (CKO); no longer LD15.2 (DOUT)
- net LD_C14: now reaches LD15.4 (CKI)
- net LD_C14: now also LD14.6 (CKO); no longer LD14.2 (DOUT)
- net LD_C41: now reaches LD42.4 (CKI)
- net LD_C41: now also LD41.6 (CKO); no longer LD41.2 (DOUT)
- net LD_C21: now reaches LD22.4 (CKI)
- net LD_C21: now also LD21.6 (CKO); no longer LD21.2 (DOUT)
- net LD_C20: now reaches LD21.4 (CKI)
- net LD_C20: now also LD20.6 (CKO); no longer LD20.2 (DOUT)
- net LD_C53: now reaches LD54.4 (CKI)
- net LD_C53: now also LD53.6 (CKO); no longer LD53.2 (DOUT)
- net LD_C52: now reaches LD53.4 (CKI)
- net LD_C52: now also LD52.6 (CKO); no longer LD52.2 (DOUT)
- net LD_C46: now reaches LD47.4 (CKI)
- net LD_C46: now also LD46.6 (CKO); no longer LD46.2 (DOUT)
- net LD_C45: now reaches LD46.4 (CKI)
- net LD_C45: now also LD45.6 (CKO); no longer LD45.2 (DOUT)
- net LD_C32: now reaches LD33.4 (CKI)
- net LD_C32: now also LD32.6 (CKO); no longer LD32.2 (DOUT)
- net LD_C10: now reaches LD11.4 (CKI)
- net LD_C10: now also LD10.6 (CKO); no longer LD10.2 (DOUT)
- net LD_C54: now reaches LD55.4 (CKI)
- net LD_C54: now also LD54.6 (CKO); no longer LD54.2 (DOUT)
- net LD_C6: now reaches LD7.4 (CKI)
- net LD_C6: now also LD6.6 (CKO); no longer LD6.2 (DOUT)
- net LD_C5: now reaches LD6.4 (CKI)
- net LD_C5: now also LD5.6 (CKO); no longer LD5.2 (DOUT)
- net LD_C36: now reaches LD37.4 (CKI)
- net LD_C36: now also LD36.6 (CKO); no longer LD36.2 (DOUT)
- net LD_C19: now reaches LD20.4 (CKI)
- net LD_C19: now also LD19.6 (CKO); no longer LD19.2 (DOUT)
- net LD_C7: now reaches LD8.4 (CKI)
- net LD_C7: now also LD7.6 (CKO); no longer LD7.2 (DOUT)
- net LD_C63: now reaches LD64.4 (CKI)
- net LD_C63: now also LD63.6 (CKO); no longer LD63.2 (DOUT)
- net LD_C47: now reaches LD48.4 (CKI)
- net LD_C47: now also LD47.6 (CKO); no longer LD47.2 (DOUT)
- net LD_C58: now reaches LD59.4 (CKI)
- net LD_C58: now also LD58.6 (CKO); no longer LD58.2 (DOUT)
- net LD_C3: now reaches LD4.4 (CKI)
- net LD_C3: now also LD3.6 (CKO); no longer LD3.2 (DOUT)
- net LD_C2: now reaches LD3.4 (CKI)
- net LD_C2: now also LD2.6 (CKO); no longer LD2.2 (DOUT)
- net LD_C40: now reaches LD41.4 (CKI)
- net LD_C40: now also LD40.6 (CKO); no longer LD40.2 (DOUT)
- net LD_C39: now reaches LD40.4 (CKI)
- net LD_C39: now also LD39.6 (CKO); no longer LD39.2 (DOUT)
- net LD_C62: now reaches LD63.4 (CKI)
- net LD_C62: now also LD62.6 (CKO); no longer LD62.2 (DOUT)
- net LD_C4: now reaches LD5.4 (CKI)
- net LD_C4: now also LD4.6 (CKO); no longer LD4.2 (DOUT)
- net LD_C1: now reaches LD2.4 (CKI)
- net LD_C1: now also LD1.6 (CKO); no longer LD1.2 (DOUT)
- net LD_C16: now reaches LD17.4 (CKI)
- net LD_C16: now also LD16.6 (CKO); no longer LD16.2 (DOUT)
- net LD_C51: now reaches LD52.4 (CKI)
- net LD_C51: now also LD51.6 (CKO); no longer LD51.2 (DOUT)
- net LD_C50: now reaches LD51.4 (CKI)
- net LD_C50: now also LD50.6 (CKO); no longer LD50.2 (DOUT)
- net LD_C49: now reaches LD50.4 (CKI)
- net LD_C49: now also LD49.6 (CKO); no longer LD49.2 (DOUT)
- net LD_C48: now reaches LD49.4 (CKI)
- net LD_C48: now also LD48.6 (CKO); no longer LD48.2 (DOUT)
- new net: LD24.1 (SDO), LD25.3 (SDI)
- new net: LD23.1 (SDO), LD24.3 (SDI)
- new net: LD31.1 (SDO), LD32.3 (SDI)
- new net: LD30.1 (SDO), LD31.3 (SDI)
- new net: LD61.1 (SDO), LD62.3 (SDI)
- new net: LD60.1 (SDO), LD61.3 (SDI)
- new net: LD57.1 (SDO), LD58.3 (SDI)
- new net: LD56.1 (SDO), LD57.3 (SDI)
- new net: LD29.1 (SDO), LD30.3 (SDI)
- new net: LD28.1 (SDO), LD29.3 (SDI)
- new net: LD26.1 (SDO), LD27.3 (SDI)
- new net: LD25.1 (SDO), LD26.3 (SDI)
- new net: LD38.1 (SDO), LD39.3 (SDI)
- new net: LD37.1 (SDO), LD38.3 (SDI)
- new net: LD13.1 (SDO), LD14.3 (SDI)
- new net: LD12.1 (SDO), LD13.3 (SDI)
- new net: LD43.1 (SDO), LD44.3 (SDI)
- new net: LD42.1 (SDO), LD43.3 (SDI)
- new net: LD27.1 (SDO), LD28.3 (SDI)
- new net: LD18.1 (SDO), LD19.3 (SDI)
- new net: LD17.1 (SDO), LD18.3 (SDI)
- new net: LD35.1 (SDO), LD36.3 (SDI)
- new net: LD34.1 (SDO), LD35.3 (SDI)
- new net: LD65.1 (SDO), LD66.3 (SDI)
- new net: LD64.1 (SDO), LD65.3 (SDI)
- new net: LD59.1 (SDO), LD60.3 (SDI)
- new net: LD10.3 (SDI), LD9.1 (SDO)
- new net: LD8.1 (SDO), LD9.3 (SDI)
- new net: LD15.1 (SDO), LD16.3 (SDI)
- new net: LD14.1 (SDO), LD15.3 (SDI)
- new net: LD41.1 (SDO), LD42.3 (SDI)
- new net: LD21.1 (SDO), LD22.3 (SDI)
- new net: LD20.1 (SDO), LD21.3 (SDI)
- new net: LD53.1 (SDO), LD54.3 (SDI)
- new net: LD52.1 (SDO), LD53.3 (SDI)
- new net: LD46.1 (SDO), LD47.3 (SDI)
- new net: LD45.1 (SDO), LD46.3 (SDI)
- new net: LD32.1 (SDO), LD33.3 (SDI)
- new net: LD10.1 (SDO), LD11.3 (SDI)
- new net: LD54.1 (SDO), LD55.3 (SDI)
- new net: LD6.1 (SDO), LD7.3 (SDI)
- new net: LD5.1 (SDO), LD6.3 (SDI)
- new net: LD36.1 (SDO), LD37.3 (SDI)
- new net: LD19.1 (SDO), LD20.3 (SDI)
- new net: LD7.1 (SDO), LD8.3 (SDI)
- new net: LD63.1 (SDO), LD64.3 (SDI)
- new net: LD47.1 (SDO), LD48.3 (SDI)
- new net: LD58.1 (SDO), LD59.3 (SDI)
- new net: LD3.1 (SDO), LD4.3 (SDI)
- new net: LD2.1 (SDO), LD3.3 (SDI)
- new net: LD40.1 (SDO), LD41.3 (SDI)
- new net: LD39.1 (SDO), LD40.3 (SDI)
- new net: LD62.1 (SDO), LD63.3 (SDI)
- new net: LD4.1 (SDO), LD5.3 (SDI)
- new net: LD1.1 (SDO), LD2.3 (SDI)
- new net: LD16.1 (SDO), LD17.3 (SDI)
- new net: LD51.1 (SDO), LD52.3 (SDI)
- new net: LD50.1 (SDO), LD51.3 (SDI)
- new net: LD49.1 (SDO), LD50.3 (SDI)
- new net: LD48.1 (SDO), LD49.3 (SDI)
- new net LC_BUF: RSC.1, U2.4 (Y)
- new net LD_C0: LD1.4 (CKI), RSC.2
- new net LD_C11: LD11.6 (CKO), LD12.4 (CKI)
- new net LD_C22: LD22.6 (CKO), LD23.4 (CKI)
- new net LD_C33: LD33.6 (CKO), LD34.4 (CKI)
- new net LD_C44: LD44.6 (CKO), LD45.4 (CKI)
- new net LD_C55: LD55.6 (CKO), LD56.4 (CKI)
- new net LED_CLK: JLB.3, U2.2 (A)
- no-connect marks 1 -> 2
Other:
- note added: "1 Data and clock entry: 3V3 -> 5 V buffers"
- note added: "2 SK9822-EC20 clocked chain, 66 pixels"
- note added: "JLB: +5V, LED_IN, LED_CLK, GND from CB1D. U1 / U2 (74AHCT1G125) buffer LED_IN / LED_CLK to 5 V logic;"
- note added: "LD_CEND_NC"
- note added: "PF233-LB1: LB1-v6 display: 66 x SK9822-EC20 clocked chain with 3V3 -> 5 V data and clock buffers"
- note added: "Pins: 1 SDO, 2 GND, 3 SDI, 4 CKI, 5 VDD (+5V), 6 CKO. LD66 SDO / CKO are left open (LD_END_NC / LD_CEND_NC)."
- note added: "RS / RSC 33 R series damping -> LD_D0 / LD_C0."
- note added: "SDO of each pixel goes straight to SDI of the next (wired); CKO -> CKI of the next by net label (LD_Cn)."
- note removed: "1 Data entry: 3V3 -> 5 V buffer"
- note removed: "2 SK6812-MINI-E chain, 66 pixels"
- note removed: "DOUT of each pixel goes straight to DIN of the next (wired); pins: 1 VDD (+5V), 2 DOUT, 3 GND, 4 DIN."
- note removed: "JLB: +5V, LED_IN, GND, GND from CB1D. U1 (74AHCT1G125) buffers LED_IN to 5 V logic; RS 33 R series damping -> LD_D0."
- note removed: "LD66 DOUT is left open (LD_END_NC)."
- note removed: "PF233-LB1: LB1 display: 66 x SK6812-MINI-E chain with 3V3 -> 5 V data buffer"
- moved on the sheet: CB, CL1, CL10, CL11, CL2, CL3, CL4, CL5, CL6, CL7, CL8, CL9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
