File: data/kicad/sch_functional/PF233-AU1_functional.kicad_sch (KiCad schematic)
At the start: 51 parts

Commit message: WIP (NOT signed off): data published by the second close-out run (8 FAIL: 3 opens on CB1D-C2 / AU1 under the exact fine-zone keep-out); third run in progress
Co-Authored-By: Claude Opus 5.5 <noreply@anthropic.com>
Claude-Session: https://claude.ai/code/session_01FX4DWSYYjMCFGGA6gmha65
Parts:
- JSWD: footprint Connector:Pin_header_1x4_P2.54mm -> Connector:Wire_pads_1x4_P2.54mm; symbol PF233F:BOX_HDR1x4 -> PF233F:BOX_WIRE1x4
Changed lines of the file:
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@@
   (wire (pts (xy 306.070 110.490) (xy 308.610 110.490)) (stroke (width 0) (type default)))
   (label "GND" (at 308.610 110.490 0) (fields_autoplaced yes) (effects (font (size 1.27 1.27)) (justify left)))
-  (symbol (lib_id "PF233F:BOX_HDR1x4") (at 332.740 116.840 0) (unit 1) (exclude_from_sim no) (in_bom yes) (on_board yes) (dnp no)
+  (symbol (lib_id "PF233F:BOX_WIRE1x4") (at 332.740 116.840 0) (unit 1) (exclude_from_sim no) (in_bom yes) (on_board yes) (dnp no)
     (property "Reference" "JSWD" (at 332.740 107.060 0) (effects (font (size 1.27 1.27))))
     (property "Value" "SWD: 3V3 SWDIO SWCLK GND" (at 332.740 127.300 0) (effects (font (size 1.0 1.0))))
-    (property "Footprint" "Connector:Pin_header_1x4_P2.54mm" (at 332.740 116.840 0) (effects (font (size 1.27 1.27)) hide))
+    (property "Footprint" "Connector:Wire_pads_1x4_P2.54mm" (at 332.740 116.840 0) (effects (font (size 1.27 1.27)) hide))
     (pin "1")
     (pin "2")

Commit message: WIP (NOT signed off): sign-off outputs with AU1 38 / 38 (exact DRC 0 / 0, all AU1 checks pass); CB1D 45 / 46 (TRIG_EXT open on the 0.125 grid, being re-routed on 0.15)
Co-Authored-By: Claude Opus 5.5 <noreply@anthropic.com>
Claude-Session: https://claude.ai/code/session_01FX4DWSYYjMCFGGA6gmha65
Parts:
- added CG1, CG2: 100n, Capacitor_SMD:C_0603_1608Metric, symbol PF233F:C_H
- added RGA, RGL: 4k7, Resistor_SMD:R_0603_1608Metric, symbol PF233F:R_H
- added RGF: 10R, Resistor_SMD:R_0603_1608Metric, symbol PF233F:R_H
- added UG: BMI270, PF233:BMI270_LGA-14_2.5x3.0mm, symbol PF233F:BOX_BMI270
Connections:
- net +3V3_AU: now also RGA.1, RGF.1, RGL.1
- net GND: now also CG1.2, CG2.2, UG.6 (GNDIO), UG.7 (GND)
- net GYR_SDA: now reaches UM.4 (PA0)
- net GYR_SDA: now also RGA.2, UG.14 (SDX)
- net GYR_SCL: now reaches UM.5 (PA1)
- net GYR_SCL: now also RGL.2, UG.13 (SCX)
- new net UG_VIO: CG1.1, CG2.1, RGF.2, UG.1 (SDO), UG.12 (CSB), UG.2 (ASDX), UG.3 (ASCX), UG.5 (VDDIO), UG.8 (VDD)
- no-connect marks 13 -> 15
Other:
- note added: "6 Yaw gyro (sweep direction, moved from CB1D)"
- note added: "PF233-AU1: AU1 audio board: descriptor link, MSPM0G3507 voice synth, TPA2005D1 speaker amp, TPA6132A2 headphone amp, 3-position output selector, BMI270 yaw gyro"
- note added: "UG BMI270 (alternate: ST LSM6DSO, same land) on I2C0, UM pins 4 / 5 (PA0 SDA / PA1 SCL); alternate address (SDO high); UG_VIO = VDD, VDDIO, CSB, SDO, pins 2 / 3,"
- note added: "UG_INT1_NC"
- note added: "UG_INT2_NC"
- note added: "UG_OCSB_NC"
- note added: "UG_OSDO_NC"
- note added: "fed from +3V3_AU by RGF 10 R with CG1 / CG2 100 nF; RGA / RGL 4k7 pull-ups. The yaw rate goes to the head in the link reply."
- note removed: "PF233-AU1: AU1 audio board: descriptor link, MSPM0G3507 voice synth, TPA2005D1 speaker amp, TPA6132A2 headphone amp, 3-position output selector"
- note removed: "UM_P4_NC"
- note removed: "UM_P5_NC"
