File: data/kicad/sch_functional/PF233-CB1D_functional.kicad_sch (KiCad schematic)
At the start: 64 parts, among them M5 5 V 1.5 A switching module, U1 Pico 2 W

Commit message: Close-out of the output modes / audio / gyro integration: sign-off 76 PASS / 0 FAIL / 4 UNVERIFIED, strict regress 114 / 0, release controls 12 / 12, publish 0 stale
AU1 (36 x 60, 8 layers, gyro moved from CB1D) routed 38 / 38, CB1D-C2 46 / 46, both exact DRC 0 / 0; PB1R-v5 AWG12 solder holes; PM2-B, HB2-B; superseded Gerber sets marked.
Tooling now default: exact-geometry DRC, router fine-pitch keep-out / neck-down / per-board grid, local repair, round checkpoints, non-destructive reset,
interface check, AU1 3-D models with gull-wing leads, counted HV check; pad check traced by the pipeline; process-guard regress row; PROCESS.md / CLAUDE.md / handoff updated.

Co-Authored-By: Claude Opus 5.5 <noreply@anthropic.com>
Claude-Session: https://claude.ai/code/session_01FX4DWSYYjMCFGGA6gmha65
Parts:
- JCL: footprint Connector:Solder_holes_AWG22_1x2_P5.08mm -> Connector:Wire_pads_AWG22_1x2_P5.08mm
- JDBG: footprint Connector:Pin_header_1x2_P2.54mm -> Connector:Wire_pads_1x2_P2.54mm
- JPB: footprint Connector:Pin_header_2x4_P2.54mm -> Connector:Wire_pads_2x4_P2.54mm
- JPW: footprint Connector:Terminal_block_1x4_P5.08mm -> Connector:Wire_pads_1x4_P5.08mm
- JTR: footprint Connector:Pin_header_1x7_P2.54mm -> Connector:Wire_pads_1x7_P2.54mm
Changed lines of the file:
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@@
     (property "Reference" "JDBG" (at 104.140 59.080 0) (effects (font (size 1.27 1.27))))
     (property "Value" "RUN / GND (reset, SWD pads on Pico underside" (at 104.140 74.240 0) (effects (font (size 1.0 1.0))))
-    (property "Footprint" "Connector:Pin_header_1x2_P2.54mm" (at 104.140 66.040 0) (effects (font (size 1.27 1.27)) hide))
+    (property "Footprint" "Connector:Wire_pads_1x2_P2.54mm" (at 104.140 66.040 0) (effects (font (size 1.27 1.27)) hide))
     (pin "1")
     (pin "2")
@@
     (property "Reference" "JPW" (at 215.900 55.880 0) (effects (font (size 1.27 1.27))))
     (property "Value" "Power in: VBUS VBUS GND GND (from shaft)" (at 215.900 76.120 0) (effects (font (size 1.0 1.0))))
-    (property "Footprint" "Connector:Terminal_block_1x4_P5.08mm" (at 215.900 66.040 0) (effects (font (size 1.27 1.27)) hide))
+    (property "Footprint" "Connector:Wire_pads_1x4_P5.08mm" (at 215.900 66.040 0) (effects (font (size 1.27 1.27)) hide))
     (pin "1")
     (pin "2")
@@
     (property "Reference" "JTR" (at 166.370 254.990 0) (effects (font (size 1.27 1.27))))
     (property "Value" "Handle: +3V3 GND TRIG DIAL AUD_LINK - SHLD" (at 166.370 280.310 0) (effects (font (size 1.0 1.0))))
-    (property "Footprint" "Connector:Pin_header_1x7_P2.54mm" (at 166.370 267.970 0) (effects (font (size 1.27 1.27)) hide))
+    (property "Footprint" "Connector:Wire_pads_1x7_P2.54mm" (at 166.370 267.970 0) (effects (font (size 1.27 1.27)) hide))
     (pin "1")
     (pin "2")
@@
     (property "Reference" "JPB" (at 39.370 361.190 0) (effects (font (size 1.27 1.27))))
     (property "Value" "to PB1R: 12V GND TX1_IN REF_I1 FAULT1_N ISEN" (at 39.370 391.590 0) (effects (font (size 1.0 1.0))))
-    (property "Footprint" "Connector:Pin_header_2x4_P2.54mm" (at 39.370 375.920 0) (effects (font (size 1.27 1.27)) hide))
+    (property "Footprint" "Connector:Wire_pads_2x4_P2.54mm" (at 39.370 375.920 0) (effects (font (size 1.27 1.27)) hide))
     (pin "1")
     (pin "2")
@@
     (property "Reference" "JCL" (at 203.200 361.190 0) (effects (font (size 1.27 1.27))))
     (property "Value" "Coil taps from TXJ1: COIL_B (drain side), CO" (at 203.200 376.350 0) (effects (font (size 1.0 1.0))))
-    (property "Footprint" "Connector:Solder_holes_AWG22_1x2_P5.08mm" (at 203.200 368.300 0) (effects (font (size 1.27 1.27)) hide))
-    (pin "1")
-    (pin "2")
+    (property "Footprint" "Connector:Wire_pads_AWG22_1x2_P5.08mm" (at 203.200 368.300 0) (effects (font (size 1.27 1.27)) hide))
+    (pin "1")
+    (pin "2")
