File: data/kicad/sch_functional/PF233-PB1R_functional.kicad_sch (KiCad schematic)
At the start: 42 parts, among them M12 12 V 1.5 A switching module, Q1A 650V SJ 95mR, Q1B 650V SJ 95mR, U1 TC4420, U3 LM393

Commit message: WIP stage 5: B3/B5/B6/B8 closed in blockers.json, B7 narrowed to HVTERM, B12 opened; cap-v18 pipeline step (cap was not regenerated on a fresh work/); upper_check septum joint by voxels; curated STLs refreshed (U6 dock for the real MT60, septum lap segments, canonical face order); DESIGN_STATE stress counts
Co-Authored-By: Claude Opus 5.5 <noreply@anthropic.com>
Claude-Session: https://claude.ai/code/session_01FX4DWSYYjMCFGGA6gmha65
Parts:
- M12: value 12 V 1.5 A switching module -> 12 V 1.0 A switching module
Changed lines of the file:
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@@
   (symbol (lib_id "PF233F:BOX_OKI3") (at 257.810 229.870 0) (unit 1) (exclude_from_sim no) (in_bom yes) (on_board yes) (dnp no)
     (property "Reference" "M12" (at 257.810 225.200 0) (effects (font (size 1.27 1.27))))
-    (property "Value" "12 V 1.5 A switching module" (at 257.810 245.110 0) (effects (font (size 1.0 1.0))))
+    (property "Value" "12 V 1.0 A switching module" (at 257.810 245.110 0) (effects (font (size 1.0 1.0))))
     (property "Footprint" "Converter_DCDC:Converter_DCDC_Murata_OKI-78SR_Horizontal" (at 257.810 229.870 0) (effects (font (size 1.27 1.27)) hide))
     (pin "1")

Commit message: WIP (NOT signed off): data published by the second close-out run (8 FAIL: 3 opens on CB1D-C2 / AU1 under the exact fine-zone keep-out); third run in progress
Co-Authored-By: Claude Opus 5.5 <noreply@anthropic.com>
Claude-Session: https://claude.ai/code/session_01FX4DWSYYjMCFGGA6gmha65
Parts:
- JC: symbol PF233F:BOX_HDR2x4 -> PF233F:BOX_WIRE2x4
- JL1: value Coil outer band: DRAIN, VBUS -> Coil pair: DRAIN1, VBUS (AWG12 soldered); footprint Connector:Terminal_block_1x2_P5.08mm -> Connector:Solder_holes_AWG12_1x2_P5.08mm; symbol PF233F:BOX_TERM2 -> PF233F:BOX_WIRE2_AWG12
- JP: symbol PF233F:BOX_TERM4 -> PF233F:BOX_WIRE4T
Changed lines of the file:
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@@
   (text "VBUS from the shaft (7S pack range 19.6 to 29.4 V) enters at JP (2 x VBUS, 2 x GND)." (exclude_from_sim no) (at 22.860 44.100 0) (effects (font (size 1.4 1.4)) (justify left top)))
   (text "Nine 100 uF 50 V hybrid cans plus four 10 uF X7R cap the DC bus of the transmit stage." (exclude_from_sim no) (at 22.860 47.300 0) (effects (font (size 1.4 1.4)) (justify left top)))
-  (symbol (lib_id "PF233F:BOX_TERM4") (at 39.370 68.580 0) (unit 1) (exclude_from_sim no) (in_bom yes) (on_board yes) (dnp no)
+  (symbol (lib_id "PF233F:BOX_WIRE4T") (at 39.370 68.580 0) (unit 1) (exclude_from_sim no) (in_bom yes) (on_board yes) (dnp no)
     (property "Reference" "JP" (at 39.370 59.080 0) (effects (font (size 1.27 1.27))))
     (property "Value" "Power in: VBUS VBUS GND GND" (at 39.370 79.320 0) (effects (font (size 1.0 1.0))))
@@
   (text "DC1 (ultrafast diode) clamps the flyback from DRAIN1 into CLAMP1: CL1A / CL1B (630 V film / C0G) with the external bleed RCL1 (5 k, lid bank)." (exclude_from_sim no) (at 223.020 141.620 0) (effects (font (size 1.4 1.4)) (justify left top)))
   (text "High-voltage nets DRAIN1 and CLAMP1: 1.0 mm clearance rule on the board." (exclude_from_sim no) (at 223.020 144.820 0) (effects (font (size 1.4 1.4)) (justify left top)))
-  (symbol (lib_id "PF233F:BOX_TERM2") (at 240.030 163.830 0) (unit 1) (exclude_from_sim no) (in_bom yes) (on_board yes) (dnp no)
+  (symbol (lib_id "PF233F:BOX_WIRE2_AWG12") (at 240.030 163.830 0) (unit 1) (exclude_from_sim no) (in_bom yes) (on_board yes) (dnp no)
     (property "Reference" "JL1" (at 240.030 156.600 0) (effects (font (size 1.27 1.27))))
-    (property "Value" "Coil outer band: DRAIN, VBUS" (at 240.030 171.760 0) (effects (font (size 1.0 1.0))))
-    (property "Footprint" "Connector:Terminal_block_1x2_P5.08mm" (at 240.030 163.830 0) (effects (font (size 1.27 1.27)) hide))
+    (property "Value" "Coil pair: DRAIN1, VBUS (AWG12 soldered)" (at 240.030 171.760 0) (effects (font (size 1.0 1.0))))
+    (property "Footprint" "Connector:Solder_holes_AWG12_1x2_P5.08mm" (at 240.030 163.830 0) (effects (font (size 1.27 1.27)) hide))
     (pin "1")
     (pin "2")
@@
   (text "JC pins: 1 SHLD, 2 GND, 3 TX1_IN, 4 REF_I1, 5 FAULT1_N, 6 ISENSE1, 7 NTC, 8 GND." (exclude_from_sim no) (at 22.860 296.080 0) (effects (font (size 1.4 1.4)) (justify left top)))
   (text "RNTC (10 k NTC on the FET spreader) -> NTC_SENSE; RUS bleeds the cable shield to GND." (exclude_from_sim no) (at 22.860 299.280 0) (effects (font (size 1.4 1.4)) (justify left top)))
-  (symbol (lib_id "PF233F:BOX_HDR2x4") (at 39.370 326.390 0) (unit 1) (exclude_from_sim no) (in_bom yes) (on_board yes) (dnp no)
+  (symbol (lib_id "PF233F:BOX_WIRE2x4") (at 39.370 326.390 0) (unit 1) (exclude_from_sim no) (in_bom yes) (on_board yes) (dnp no)
     (property "Reference" "JC" (at 39.370 311.060 0) (effects (font (size 1.27 1.27))))
     (property "Value" "Umbilical from the head: SHLD GND TX1_IN REF" (at 39.370 341.460 0) (effects (font (size 1.0 1.0))))

Commit message: Close-out of the output modes / audio / gyro integration: sign-off 76 PASS / 0 FAIL / 4 UNVERIFIED, strict regress 114 / 0, release controls 12 / 12, publish 0 stale
AU1 (36 x 60, 8 layers, gyro moved from CB1D) routed 38 / 38, CB1D-C2 46 / 46, both exact DRC 0 / 0; PB1R-v5 AWG12 solder holes; PM2-B, HB2-B; superseded Gerber sets marked.
Tooling now default: exact-geometry DRC, router fine-pitch keep-out / neck-down / per-board grid, local repair, round checkpoints, non-destructive reset,
interface check, AU1 3-D models with gull-wing leads, counted HV check; pad check traced by the pipeline; process-guard regress row; PROCESS.md / CLAUDE.md / handoff updated.

Co-Authored-By: Claude Opus 5.5 <noreply@anthropic.com>
Claude-Session: https://claude.ai/code/session_01FX4DWSYYjMCFGGA6gmha65
Parts:
- JC: footprint Connector:Pin_header_2x4_P2.54mm -> Connector:Wire_pads_2x4_P2.54mm
- JL1: footprint Connector:Solder_holes_AWG12_1x2_P5.08mm -> Connector:Wire_pads_AWG12_1x2_P5.08mm
- JP: footprint Connector:Terminal_block_1x4_P5.08mm -> Connector:Wire_pads_1x4_P5.08mm
Changed lines of the file:
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@@
     (property "Reference" "JP" (at 39.370 59.080 0) (effects (font (size 1.27 1.27))))
     (property "Value" "Power in: VBUS VBUS GND GND" (at 39.370 79.320 0) (effects (font (size 1.0 1.0))))
-    (property "Footprint" "Connector:Terminal_block_1x4_P5.08mm" (at 39.370 68.580 0) (effects (font (size 1.27 1.27)) hide))
+    (property "Footprint" "Connector:Wire_pads_1x4_P5.08mm" (at 39.370 68.580 0) (effects (font (size 1.27 1.27)) hide))
     (pin "1")
     (pin "2")
@@
     (property "Reference" "JL1" (at 240.030 156.600 0) (effects (font (size 1.27 1.27))))
     (property "Value" "Coil pair: DRAIN1, VBUS (AWG12 soldered)" (at 240.030 171.760 0) (effects (font (size 1.0 1.0))))
-    (property "Footprint" "Connector:Solder_holes_AWG12_1x2_P5.08mm" (at 240.030 163.830 0) (effects (font (size 1.27 1.27)) hide))
+    (property "Footprint" "Connector:Wire_pads_AWG12_1x2_P5.08mm" (at 240.030 163.830 0) (effects (font (size 1.27 1.27)) hide))
     (pin "1")
     (pin "2")
@@
     (property "Reference" "JC" (at 39.370 311.060 0) (effects (font (size 1.27 1.27))))
     (property "Value" "Umbilical from the head: SHLD GND TX1_IN REF" (at 39.370 341.460 0) (effects (font (size 1.0 1.0))))
-    (property "Footprint" "Connector:Pin_header_2x4_P2.54mm" (at 39.370 326.390 0) (effects (font (size 1.27 1.27)) hide))
-    (pin "1")
-    (pin "2")
+    (property "Footprint" "Connector:Wire_pads_2x4_P2.54mm" (at 39.370 326.390 0) (effects (font (size 1.27 1.27)) hide))
+    (pin "1")
+    (pin "2")

Commit message: WIP: published PB1R KiCad / schematic outputs and pipeline graph for the B7 close-out (sign-off re-run pending)
Co-Authored-By: Claude Opus 5.5 <noreply@anthropic.com>
Claude-Session: https://claude.ai/code/session_01FX4DWSYYjMCFGGA6gmha65
Parts:
- RCL1: value external 5k 10W (lid bank) -> 4 x Vishay PR03 1K24 1% 750V 3W in series, 4
Other:
- note added: "DC1 (ultrafast diode) clamps the flyback from DRAIN1 into CLAMP1: CL1A / CL1B (630 V film / C0G) with the external bleed RCL1 (4 x Vishay PR03 1K24 in series, 4.96 k, potted in the NPM hot zone)."
- note removed: "DC1 (ultrafast diode) clamps the flyback from DRAIN1 into CLAMP1: CL1A / CL1B (630 V film / C0G) with the external bleed RCL1 (5 k, lid bank)."
Changed lines of the file:
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@@
-(kicad_sch (version 20231120) (generator "arx_sch_func") (generator_version "1") (paper "User" 482.6 406.4)
+(kicad_sch (version 20231120) (generator "arx_sch_func") (generator_version "1") (paper "User" 508.0 406.4)
   (title_block (title "PF233-PB1R  functional schematic") (date "2026-10-26") (rev "r3") (company "ARX / PHI-FOLD 233") (comment 1 "PB1R transmit stage: gate drive, two 650 V FETs, shunt, flyback clamp, overcurrent comparator, 12 V aux") (comment 2 "MODELED design: not built, not bench-tested.") (comment 3 "Generated: src/pcb/sch_func.py; checked against the netlist."))
   (text "How to read: parts sit in functional blocks (dashed frames). Every pin ends in a short wire with its NET NAME; equal names are connected (also between blocks). A cross = intentionally unconnected pin." (exclude_from_sim no) (at 20.320 10.160 0) (effects (font (size 1.4 1.4)) (justify left top)))
@@
   (wire (pts (xy 195.580 157.480) (xy 198.120 157.480)) (stroke (width 0) (type default)))
   (label "GND" (at 198.120 157.480 0) (fields_autoplaced yes) (effects (font (size 1.27 1.27)) (justify left)))
-  (rectangle (start 220.48 132.42) (end 407.94 178.34) (stroke (width 0.3) (type dash)) (fill (type none)))
+  (rectangle (start 220.48 132.42) (end 472.23 178.34) (stroke (width 0.3) (type dash)) (fill (type none)))
   (text "4  Coil connection and flyback clamp" (exclude_from_sim no) (at 223.020 134.420 0) (effects (font (size 2.54 2.54) bold) (justify left top)))
   (text "JL1: coil outer band between DRAIN1 and VBUS." (exclude_from_sim no) (at 223.020 138.420 0) (effects (font (size 1.4 1.4)) (justify left top)))
-  (text "DC1 (ultrafast diode) clamps the flyback from DRAIN1 into CLAMP1: CL1A / CL1B (630 V film / C0G) with the external bleed RCL1 (5 k, lid bank)." (exclude_from_sim no) (at 223.020 141.620 0) (effects (font (size 1.4 1.4)) (justify left top)))
+  (text "DC1 (ultrafast diode) clamps the flyback from DRAIN1 into CLAMP1: CL1A / CL1B (630 V film / C0G) with the external bleed RCL1 (4 x Vishay PR03 1K24 in series, 4.96 k, potted in the NPM hot zone)." (exclude_from_sim no) (at 223.020 141.620 0) (effects (font (size 1.4 1.4)) (justify left top)))
   (text "High-voltage nets DRAIN1 and CLAMP1: 1.0 mm clearance rule on the board." (exclude_from_sim no) (at 223.020 144.820 0) (effects (font (size 1.4 1.4)) (justify left top)))
   (symbol (lib_id "PF233F:BOX_WIRE2_AWG12") (at 240.030 163.830 0) (unit 1) (exclude_from_sim no) (in_bom yes) (on_board yes) (dnp no)
@@
   (symbol (lib_id "PF233F:BOX_WIRE2") (at 381.000 163.830 0) (unit 1) (exclude_from_sim no) (in_bom yes) (on_board yes) (dnp no)
     (property "Reference" "RCL1" (at 381.000 156.600 0) (effects (font (size 1.27 1.27))))
-    (property "Value" "external 5k 10W (lid bank)" (at 381.000 171.760 0) (effects (font (size 1.0 1.0))))
+    (property "Value" "4 x Vishay PR03 1K24 1% 750V 3W in series, 4" (at 381.000 171.760 0) (effects (font (size 1.0 1.0))))
     (property "Footprint" "Connector:SolderPad_2x_P5.08mm" (at 381.000 163.830 0) (effects (font (size 1.27 1.27)) hide))
     (pin "1")

Commit message: Speed-up: batched Gerber geometry (10x, same copper) and parallel sign-off controls (245 s -> 32 s); B7 sign-off run
gerber_geom.layer_geometry merges same-polarity runs with unary_union (worst sym-diff 6e-13 mm2
over 258 layers; regress row keeps the sequential build as reference). publish 79 -> 10.5 s.
release_signoff_controls runs independent jobs in a thread pool, stale-data control alone last.
Sign-off 77 PASS / 0 FAIL / 3 UNVERIFIED, strict regress 120 / 0, publish 0 stale.
Moved: US3M diode margins (reverse voltage 27.5 -> 56.5 %, current 80.1 -> 83.4 %).

Co-Authored-By: Claude Opus 5.5 <noreply@anthropic.com>
Claude-Session: https://claude.ai/code/session_01FX4DWSYYjMCFGGA6gmha65
Parts:
- DC1: value ES3J 600V 3A -> US3M 1000V 3A
Changed lines of the file:
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@@
   (symbol (lib_id "PF233F:D_H") (at 281.940 160.020 0) (unit 1) (exclude_from_sim no) (in_bom yes) (on_board yes) (dnp no)
     (property "Reference" "DC1" (at 281.940 157.020 0) (effects (font (size 1.27 1.27))))
-    (property "Value" "ES3J 600V 3A" (at 281.940 163.020 0) (effects (font (size 1.0 1.0))))
+    (property "Value" "US3M 1000V 3A" (at 281.940 163.020 0) (effects (font (size 1.0 1.0))))
     (property "Footprint" "Diode_SMD:D_SMC" (at 281.940 160.020 0) (effects (font (size 1.27 1.27)) hide))
     (pin "2")
