File: data/kicad/sch/PF233-HB2.kicad_sch (KiCad schematic)
At the start: 10 parts

Commit message: Step 5: datasheets and fabricator sheets (vendor-derived floor, verified parts, PB1R 9-can bank, Gerber edge read-back)
- Fab floor from AdvancedPCB / TTM pages (docs/design/FAB_RULES_VERIFIED.md, U-FAB-RULES closed): clearance 0.16,
  component-PTH ring 0.18 / hole 0.46, drill-copper 0.26, drill-drill 0.41, every rule (severity error).
  CB1D JA/JB and HB2 TO-92 pads 1.02 mm; route_fix merges close same-net vias (CB1D, LB1).
- Parts from manufacturer PDFs (docs/design/DATASHEET_LOG.md): PB1R bulk 9 x Panasonic EEHZC1H101P
  (the 150 uF / 50 V polymer-Ta was not found; bank stays 900 uF, on-time table unchanged), PB1R re-placed
  with the Kelvin/comparator cluster pinned (pulse path 4.9 mohm, spike 7.5 V, ground ref 15.5 mV unchanged);
  SMCJ30A (SMCJ33A clamps 53.3 V > 50 V parts), Si4401FDY, BZT52C15, Bourns SF-1206S500-2 (new 1206 land),
  DRV5023BIQLPG, CRCW2512 500 V, OPA2365/OPA2211/LM393/CD74HC4051 checked. ES3J 600 V kept as a WATCH.
- U-DS-PARTS split into groups; open: TXDRIVE, OKI, PACK, BAV199, HVTERM. U-COLD-BOOTSTRAP closed.
- Controls retargeted to fixture folders (12/12). Netlist date fixed (data changed daily).
- Gerber planes from gerber_out.py ran into the notch and to 0.1 mm of the edge since r1 (found by the
  independent review): fixed, and gerber_edge_check.py reads every copper layer back.
- New Gerber sets CB1D_B3, LB1_v5, PB1R_v2; old sets marked SUPERSEDED.
- Findings for the owner: aluminium cans ~0.5 x a 1 g nugget (OPEN_ITEMS 34), OPA2365 capacitive load (30),
  OPA2211 input range on 5 V (31), Hall magnet spread (32).
- Strict regress 55 PASS / 0 FAIL / 0 SKIP; sign-off 44 PASS / 0 FAIL / 0 SKIP / 19 UNVERIFIED.

Co-Authored-By: Claude Opus 5.5 <noreply@anthropic.com>
Claude-Session: https://claude.ai/code/session_015VKhZtgEAWnezB2NDY75VV
Parts:
- HS1: value Hall switch OD -> DRV5023BIQLPG
Changed lines of the file:
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@@
   (symbol (lib_id "PF233_auto:HS1") (at 30.48 40.64 0) (unit 1) (exclude_from_sim no) (in_bom yes) (on_board yes) (dnp no)
     (property "Reference" "HS1" (at 30.48 38.10 0) (effects (font (size 1.27 1.27))))
-    (property "Value" "Hall switch OD" (at 30.48 46.99 0) (effects (font (size 1.0 1.0))))
+    (property "Value" "DRV5023BIQLPG" (at 30.48 46.99 0) (effects (font (size 1.0 1.0))))
     (property "Footprint" "Package_TO_SOT_THT:TO-92_Inline" (at 30.48 40.64 0) (effects (font (size 1.27 1.27)) hide))
     (pin "1")

Commit message: WIP (NOT signed off): data published by the first close-out sign-off run, which had 5 FAIL (CB1D-C2 / AU1 fine-pitch clearance); superseded by the rerun in progress
Co-Authored-By: Claude Opus 5.5 <noreply@anthropic.com>
Claude-Session: https://claude.ai/code/session_01FX4DWSYYjMCFGGA6gmha65
Parts:
- added JAU: Lead to AU1: AUD_LINK, GND, Connector:SolderPad_2x_P5.08mm, symbol PF233_auto:JAU
Connections:
- net GND: now also JAU.2
- net JH5_NC renamed AUD_LINK
- net AUD_LINK: now also JAU.1
Other:
- moved on the sheet: JDIAL, JH, RD0, RD2, RD3, RD4, RH1, RSHH

Commit message: Close-out of the output modes / audio / gyro integration: sign-off 76 PASS / 0 FAIL / 4 UNVERIFIED, strict regress 114 / 0, release controls 12 / 12, publish 0 stale
AU1 (36 x 60, 8 layers, gyro moved from CB1D) routed 38 / 38, CB1D-C2 46 / 46, both exact DRC 0 / 0; PB1R-v5 AWG12 solder holes; PM2-B, HB2-B; superseded Gerber sets marked.
Tooling now default: exact-geometry DRC, router fine-pitch keep-out / neck-down / per-board grid, local repair, round checkpoints, non-destructive reset,
interface check, AU1 3-D models with gull-wing leads, counted HV check; pad check traced by the pipeline; process-guard regress row; PROCESS.md / CLAUDE.md / handoff updated.

Co-Authored-By: Claude Opus 5.5 <noreply@anthropic.com>
Claude-Session: https://claude.ai/code/session_01FX4DWSYYjMCFGGA6gmha65
Parts:
- JDIAL: footprint Connector:Pin_header_1x5_P2.54mm -> Connector:Wire_pads_1x5_P2.54mm
- JH: footprint Connector:Pin_header_1x7_P2.54mm -> Connector:Wire_pads_1x7_P2.54mm
Changed lines of the file:
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@@
     (property "Reference" "JDIAL" (at 30.48 60.96 0) (effects (font (size 1.27 1.27))))
     (property "Value" "Dial: COM P1 P2 P3 P4 (4-pos rotary, top housing)" (at 30.48 72.39 0) (effects (font (size 1.0 1.0))))
-    (property "Footprint" "Connector:Pin_header_1x5_P2.54mm" (at 30.48 63.50 0) (effects (font (size 1.27 1.27)) hide))
+    (property "Footprint" "Connector:Wire_pads_1x5_P2.54mm" (at 30.48 63.50 0) (effects (font (size 1.27 1.27)) hide))
     (pin "1")
     (pin "2")
@@
     (property "Reference" "JH" (at 30.48 76.20 0) (effects (font (size 1.27 1.27))))
     (property "Value" "Signal cord to the head: +3V3 GND TRIG DIAL - - SHLD" (at 30.48 90.17 0) (effects (font (size 1.0 1.0))))
-    (property "Footprint" "Connector:Pin_header_1x7_P2.54mm" (at 30.48 78.74 0) (effects (font (size 1.27 1.27)) hide))
+    (property "Footprint" "Connector:Wire_pads_1x7_P2.54mm" (at 30.48 78.74 0) (effects (font (size 1.27 1.27)) hide))
     (pin "1")
     (pin "2")
